Commit message: add namespace

File: Scout_mini_ROS1_Navigation/scout_gazebo_sim/scout/scout_description/urdf/gps.xacro (robot description, xacro)
@@ -3,6 +3,6 @@
 <!-- https://classic.gazebosim.org/tutorials?tut=ros_gzplugins#Camera -->
 <robot xmlns:xacro="http://ros.org/wiki/xacro" name="scout_camera">
-    <xacro:macro name="GPS" params="parent_link *joint_pose">
-        <xacro:property name="topicName"    default="/gps" />
+    <xacro:macro name="GPS" params="parent_link *joint_pose topic_name:=/gps">
+        <xacro:property name="topicName"    default="${topic_name}" />
         <joint name="gps_joint" type="fixed">
             <axis xyz="0 1 0" />

File: Scout_mini_ROS1_Navigation/scout_gazebo_sim/scout/scout_description/urdf/hokuyo_2d.xacro (robot description, xacro)
@@ -3,6 +3,6 @@
 <!-- https://classic.gazebosim.org/tutorials?tut=ros_gzplugins#GPULaser -->
 <robot xmlns:xacro="http://ros.org/wiki/xacro" name="scout_lidar">
-    <xacro:macro name="hokuyo_lidar" params="parent_link visualize:=false *joint_pose gpu:=false">
-        <xacro:property name="topicName"    default="/hokuyo/scan" />
+    <xacro:macro name="hokuyo_lidar" params="parent_link visualize:=false *joint_pose gpu:=false topic_name:=/hokuyo/scan">
+        <xacro:property name="topicName"    default="${topic_name}" />
         <xacro:property name="samples"      default="720"          />
         <xacro:property name="min_range"    default="0.10"         />

File: Scout_mini_ROS1_Navigation/scout_gazebo_sim/scout/scout_description/urdf/mini.xacro (robot description, xacro)
@@ -177,5 +177,5 @@
     <xacro:if value="$(arg hokuyo_lidar)" >
         <xacro:include filename="$(find scout_description)/urdf/hokuyo_2d.xacro" />
-        <xacro:hokuyo_lidar parent_link="base_link" visualize="$(arg visualize)" gpu="${gpu}">
+        <xacro:hokuyo_lidar parent_link="base_link" visualize="$(arg visualize)" gpu="${gpu}" topic_name="/$(arg robot_namespace)/hokuyo/scan">
             <origin xyz="${lidar_pose}" rpy="${lidar_orientation}" />
         </xacro:hokuyo_lidar>
@@ -189,5 +189,5 @@
     <xacro:if value="$(arg camera)" >
         <xacro:include filename="$(find scout_description)/urdf/$(arg camera_name).xacro" />
-        <xacro:scout_camera parent_link="base_link" name="camera" topics_ns="camera" publish_pointcloud="$(arg camera_pointcloud)" visualize="$(arg visualize)" xyz="${camera_pose}" rpy="${camera_orientation}" />
+        <xacro:scout_camera parent_link="base_link" name="camera" topics_ns="$(arg robot_namespace)/camera" publish_pointcloud="$(arg camera_pointcloud)" visualize="$(arg visualize)" xyz="${camera_pose}" rpy="${camera_orientation}" />
     </xacro:if>
     <!-- IMU -->
@@ -201,5 +201,5 @@
     <xacro:if value="$(arg gps)" >
         <xacro:include filename="$(find scout_description)/urdf/gps.xacro" />
-        <xacro:GPS parent_link="base_link" >
+        <xacro:GPS parent_link="base_link" topic_name="/$(arg robot_namespace)/gps" >
             <origin xyz="${gps_pose}" rpy="${gps_orientation}" />
         </xacro:GPS>

File: Scout_mini_ROS1_Navigation/scout_gazebo_sim/scout/scout_description/urdf/realsense-d435.xacro (robot description, xacro)
@@ -5,5 +5,5 @@
     <xacro:macro name="scout_camera" params="parent_link name topics_ns:=camera publish_pointcloud:=false visualize:=false xyz rpy">
     <xacro:include filename="$(find scout_description)/urdf/_d435.urdf.xacro" />
-    <xacro:sensor_d435 parent="${parent_link}" name="camera" topics_ns="camera" publish_pointcloud="$(arg camera_pointcloud)" visualize="$(arg visualize)">
+    <xacro:sensor_d435 parent="${parent_link}" name="${name}" topics_ns="${topics_ns}" publish_pointcloud="${publish_pointcloud}" visualize="${visualize}">
         <origin xyz="${xyz}" rpy="${rpy}" />
     </xacro:sensor_d435>
