Commit message: 强制更改imu_link的命名空间

File: Scout_mini_ROS1_Navigation/scout_gazebo_sim/scout/scout_description/urdf/imu.xacro (robot description, xacro)
@@ -3,6 +3,5 @@
 <!-- https://classic.gazebosim.org/tutorials?tut=ros_gzplugins#GPULaser -->
 <robot xmlns:xacro="http://ros.org/wiki/xacro" name="scout_imu">
-    <xacro:arg name="robot_namespace" default="/" />
-    <xacro:macro name="IMU" params="parent_link *joint_pose">
+    <xacro:macro name="IMU" params="parent_link imu_frame *joint_pose">
         <xacro:property name="topicName"    default="/imu" />
         <link name="imu_link">
@@ -45,5 +44,5 @@
                     <xyzOffset>0 0 0</xyzOffset>
                     <rpyOffset>0 0 0</rpyOffset>
-                    <frameName>$(arg robot_namespace)/imu_link</frameName>
+                    <frameName>${imu_frame}</frameName>
                     <initialOrientationAsReference>false</initialOrientationAsReference>
                 </plugin>

File: Scout_mini_ROS1_Navigation/scout_gazebo_sim/scout/scout_description/urdf/mini.xacro (robot description, xacro)
@@ -8,4 +8,5 @@
     <xacro:arg name="camera"    default="true"      />
     <xacro:arg name="imu"       default="true"      />
+    <xacro:arg name="imu_frame" default="imu_link"  />
     <xacro:arg name="gps"       default="true"      />
     <xacro:arg name="visualize" default="false"     />
@@ -194,5 +195,5 @@
     <xacro:if value="$(arg imu)" >
         <xacro:include filename="$(find scout_description)/urdf/imu.xacro" />
-        <xacro:IMU parent_link="base_link" >
+        <xacro:IMU parent_link="base_link" imu_frame="$(arg imu_frame)">
             <origin xyz="${imu_pose}" rpy="${imu_orientation}" />
         </xacro:IMU>
