Commit message: Fix: Scout AMCL scan topic and Go2 lidar namespace issues
- Fix Scout AMCL scan_topic to use full namespace path /robot_X/hokuyo/scan
- Fix Go2 lidar topic namespace duplication by using robotNamespace parameter
- Resolve TF and topic namespace conflicts in multi-robot setup
- Add new launch files and multi-robot support

File: scout_mini/scout_gazebo_sim/scout/scout_description/urdf/gps.xacro (robot description, xacro)
@@ -3,5 +3,5 @@
 <!-- https://classic.gazebosim.org/tutorials?tut=ros_gzplugins#Camera -->
 <robot xmlns:xacro="http://ros.org/wiki/xacro" name="scout_camera">
-    <xacro:macro name="GPS" params="parent_link *joint_pose topic_name:=/gps">
+    <xacro:macro name="GPS" params="parent_link *joint_pose robot_namespace:='' topic_name:='gps'">
         <xacro:property name="topicName"    default="${topic_name}" />
         <joint name="gps_joint" type="fixed">
@@ -34,4 +34,5 @@
         <gazebo>
             <plugin name="gazebo_ros_gps" filename="libhector_gazebo_ros_gps.so">
+                <robotNamespace>${robot_namespace}</robotNamespace>
                 <updateRate>4.0</updateRate>
                 <bodyName>${parent_link}</bodyName>

File: scout_mini/scout_gazebo_sim/scout/scout_description/urdf/hokuyo_2d.xacro (robot description, xacro)
@@ -3,6 +3,8 @@
 <!-- https://classic.gazebosim.org/tutorials?tut=ros_gzplugins#GPULaser -->
 <robot xmlns:xacro="http://ros.org/wiki/xacro" name="scout_lidar">
-    <xacro:macro name="hokuyo_lidar" params="parent_link visualize:=false *joint_pose gpu:=false topic_name:=/hokuyo/scan">
+    <xacro:macro name="hokuyo_lidar" params="parent_link visualize:=false *joint_pose gpu:=false robot_namespace:='' topic_name:=/hokuyo/scan">
         <xacro:property name="topicName"    default="${topic_name}" />
+        <xacro:property name="frameName"   default="${robot_namespace}/hokuyo_link" if="${robot_namespace}" />
+        <xacro:property name="frameName"   default="hokuyo_link" unless="${robot_namespace}" />
         <xacro:property name="samples"      default="720"          />
         <xacro:property name="min_range"    default="0.10"         />
@@ -71,6 +73,7 @@
                 <!-- <plugin name="gazebo_ros_head_hokuyo_controller" filename="libgazebo_ros_laser.so"> -->
                 <plugin name="gazebo_ros_head_hokuyo_controller" filename="libgazebo_ros_gpu_laser.so">
+                    <robotNamespace>${robot_namespace}</robotNamespace>
                     <topicName>${topicName}</topicName>
-                    <frameName>hokuyo_link</frameName>
+                    <frameName>${frameName}</frameName>
                 </plugin>
                 </sensor>
@@ -113,6 +116,7 @@
                 <!-- <plugin name="gazebo_ros_head_hokuyo_controller" filename="libgazebo_ros_laser.so"> -->
                 <plugin name="gazebo_ros_head_hokuyo_controller" filename="libgazebo_ros_laser.so">
+                    <robotNamespace>${robot_namespace}</robotNamespace>
                     <topicName>${topicName}</topicName>
-                    <frameName>hokuyo_link</frameName>
+                    <frameName>${frameName}</frameName>
                 </plugin>
                 </sensor>

File: scout_mini/scout_gazebo_sim/scout/scout_description/urdf/imu.xacro (robot description, xacro)
@@ -3,6 +3,8 @@
 <!-- https://classic.gazebosim.org/tutorials?tut=ros_gzplugins#GPULaser -->
 <robot xmlns:xacro="http://ros.org/wiki/xacro" name="scout_imu">
-    <xacro:macro name="IMU" params="parent_link imu_frame *joint_pose">
-        <xacro:property name="topicName"    default="/imu" />
+    <xacro:macro name="IMU" params="parent_link imu_frame *joint_pose robot_namespace:='' topic_name:='imu'">
+        <xacro:property name="topicName"    default="${topic_name}" />
+        <xacro:property name="frameName"   default="${robot_namespace}/${imu_frame}" if="${robot_namespace}" />
+        <xacro:property name="frameName"   default="${imu_frame}" unless="${robot_namespace}" />
         <link name="imu_link">
             <inertial>
@@ -38,4 +40,5 @@
                 <topic>__default_topic__</topic>
                 <plugin filename="libgazebo_ros_imu_sensor.so" name="imu_plugin">
+                    <robotNamespace>${robot_namespace}</robotNamespace>
                     <topicName>${topicName}</topicName>
                     <bodyName>imu_link</bodyName>
@@ -44,5 +47,5 @@
                     <xyzOffset>0 0 0</xyzOffset>
                     <rpyOffset>0 0 0</rpyOffset>
-                    <frameName>${imu_frame}</frameName>
+                    <frameName>${frameName}</frameName>
                     <initialOrientationAsReference>false</initialOrientationAsReference>
                 </plugin>

File: scout_mini/scout_gazebo_sim/scout/scout_description/urdf/mini.xacro (robot description, xacro)
@@ -1,5 +1,5 @@
 <?xml version="1.0"?>
 <robot name="scout_mini" xmlns:xacro="http://ros.org/wiki/xacro">
-    <xacro:arg name="robot_namespace" default="/" />
+    <xacro:arg name="robot_namespace" default="" />
     <xacro:arg name="urdf_extras" default="empty.urdf" />
     <!-- Sensors Configuration -->
@@ -178,5 +178,5 @@
     <xacro:if value="$(arg hokuyo_lidar)" >
         <xacro:include filename="$(find scout_description)/urdf/hokuyo_2d.xacro" />
-        <xacro:hokuyo_lidar parent_link="base_link" visualize="$(arg visualize)" gpu="${gpu}" topic_name="/$(arg robot_namespace)/hokuyo/scan">
+        <xacro:hokuyo_lidar parent_link="base_link" visualize="$(arg visualize)" gpu="${gpu}" robot_namespace="$(arg robot_namespace)" topic_name="hokuyo/scan">
             <origin xyz="${lidar_pose}" rpy="${lidar_orientation}" />
         </xacro:hokuyo_lidar>
@@ -190,10 +190,10 @@
     <xacro:if value="$(arg camera)" >
         <xacro:include filename="$(find scout_description)/urdf/$(arg camera_name).xacro" />
-        <xacro:scout_camera parent_link="base_link" name="camera" topics_ns="$(arg robot_namespace)/camera" publish_pointcloud="$(arg camera_pointcloud)" visualize="$(arg visualize)" xyz="${camera_pose}" rpy="${camera_orientation}" />
+        <xacro:scout_camera parent_link="base_link" name="camera" topics_ns="camera" publish_pointcloud="$(arg camera_pointcloud)" visualize="$(arg visualize)" xyz="${camera_pose}" rpy="${camera_orientation}" />
     </xacro:if>
     <!-- IMU -->
     <xacro:if value="$(arg imu)" >
         <xacro:include filename="$(find scout_description)/urdf/imu.xacro" />
-        <xacro:IMU parent_link="base_link" imu_frame="$(arg imu_frame)">
+        <xacro:IMU parent_link="base_link" imu_frame="$(arg imu_frame)" robot_namespace="$(arg robot_namespace)" topic_name="imu">
             <origin xyz="${imu_pose}" rpy="${imu_orientation}" />
         </xacro:IMU>
@@ -202,5 +202,5 @@
     <xacro:if value="$(arg gps)" >
         <xacro:include filename="$(find scout_description)/urdf/gps.xacro" />
-        <xacro:GPS parent_link="base_link" topic_name="/$(arg robot_namespace)/gps" >
+        <xacro:GPS parent_link="base_link" robot_namespace="$(arg robot_namespace)" topic_name="gps">
             <origin xyz="${gps_pose}" rpy="${gps_orientation}" />
         </xacro:GPS>

File: unitree_go2/unitree_ros/robots/go2_description/xacro/robot.xacro (robot description, xacro)
@@ -90,5 +90,5 @@
     </link>
     <!--模型好一点的2d激光雷达-->
-<!--配置雷达简易版，使用圆柱体表示-->
+    <!--配置雷达简易版，使用圆柱体表示-->
     <link name="lidar">
         <visual>
