Commit message: 自己的配置

File: scout_mini/scout_gazebo_sim/scout/scout_description/urdf/hokuyo_2d.xacro (robot description, xacro)
@@ -5,6 +5,7 @@
     <xacro:macro name="hokuyo_lidar" params="parent_link visualize:=false *joint_pose gpu:=false robot_namespace:='' topic_name:=/hokuyo/scan">
         <xacro:property name="topicName"    default="${topic_name}" />
-        <xacro:property name="frameName"   default="${robot_namespace}/hokuyo_link" if="${robot_namespace}" />
-        <xacro:property name="frameName"   default="hokuyo_link" unless="${robot_namespace}" />
+        <!-- frameName should be just the link name without namespace prefix -->
+        <!-- The tf_prefix in robot_state_publisher will automatically add the namespace prefix -->
+        <xacro:property name="frameName"   default="hokuyo_link" />
         <xacro:property name="samples"      default="720"          />
         <xacro:property name="min_range"    default="0.10"         />

File: scout_mini/scout_gazebo_sim/scout/scout_description/urdf/imu.xacro (robot description, xacro)
@@ -3,6 +3,12 @@
 <!-- https://classic.gazebosim.org/tutorials?tut=ros_gzplugins#GPULaser -->
 <robot xmlns:xacro="http://ros.org/wiki/xacro" name="scout_imu">
-    <xacro:macro name="IMU" params="parent_link imu_frame *joint_pose robot_namespace:='' topic_name:='imu'">
+    <xacro:macro name="IMU" params="parent_link imu_frame *joint_pose robot_namespace:='' topic_namespace:='' topic_name:='imu'">
         <xacro:property name="topicName"    default="${topic_name}" />
+        <!-- Use topic_namespace for robotNamespace (for topics), robot_namespace for frameName (for TF frames) -->
+        <!-- If topic_namespace is not provided, fall back to robot_namespace for backward compatibility -->
+        <xacro:property name="topicNamespace" default="${topic_namespace}" if="${topic_namespace}" />
+        <xacro:property name="topicNamespace" default="${robot_namespace}" unless="${topic_namespace}" />
+        <!-- frameName for IMU message frame_id: needs to include namespace prefix to match TF frames -->
+        <!-- This is different from TF frame names - IMU message frame_id must match the actual TF frame name -->
         <xacro:property name="frameName"   default="${robot_namespace}/${imu_frame}" if="${robot_namespace}" />
         <xacro:property name="frameName"   default="${imu_frame}" unless="${robot_namespace}" />
@@ -40,5 +46,5 @@
                 <topic>__default_topic__</topic>
                 <plugin filename="libgazebo_ros_imu_sensor.so" name="imu_plugin">
-                    <robotNamespace>${robot_namespace}</robotNamespace>
+                    <!-- <robotNamespace>${topicNamespace}</robotNamespace> -->
                     <topicName>${topicName}</topicName>
                     <bodyName>imu_link</bodyName>

File: scout_mini/scout_gazebo_sim/scout/scout_description/urdf/mini.xacro (robot description, xacro)
@@ -195,5 +195,6 @@
     <xacro:if value="$(arg imu)" >
         <xacro:include filename="$(find scout_description)/urdf/imu.xacro" />
-        <xacro:IMU parent_link="base_link" imu_frame="$(arg imu_frame)" robot_namespace="$(arg robot_namespace)" topic_name="imu">
+        <!-- Explicitly pass topic_namespace to ensure IMU publishes to /robot_X/imu -->
+        <xacro:IMU parent_link="base_link" imu_frame="$(arg imu_frame)" robot_namespace="$(arg robot_namespace)" topic_namespace="$(arg robot_namespace)" topic_name="imu">
             <origin xyz="${imu_pose}" rpy="${imu_orientation}" />
         </xacro:IMU>

File: unitree_go2/unitree_ros/robots/go2_description/xacro/gazebo.xacro (robot description, xacro)
@@ -43,6 +43,6 @@
             <topic>__default_topic__</topic>
             <plugin filename="libgazebo_ros_imu_sensor.so" name="imu_plugin">
-                <robotNamespace>$(arg robot_namespace)</robotNamespace>
-                <topicName>trunk_imu</topicName>
+                <!-- <robotNamespace>$(arg robot_namespace)</robotNamespace> -->
+                <topicName>go2_gazebo/trunk_imu</topicName>
                 <bodyName>imu_link</bodyName>
                 <updateRateHZ>1000.0</updateRateHZ>
@@ -50,5 +50,6 @@
                 <xyzOffset>0 0 0</xyzOffset>
                 <rpyOffset>0 0 0</rpyOffset>
-                <frameName>imu_link</frameName>
+                <frameName>go2_gazebo/imu_link</frameName>
+                <!-- <frameName>imu_link</frameName> -->
             </plugin>
             <pose>0 0 0 0 0 0</pose>
@@ -82,7 +83,7 @@
             </ray>
             <plugin name="gazebo_ros_hokuyo_controller" filename="libgazebo_ros_laser.so">
-                <robotNamespace>$(arg robot_namespace)</robotNamespace>
-                <topicName>scan</topicName>
-                <frameName>$(arg robot_namespace)/lidar</frameName>
+                <!-- <robotNamespace>$(arg robot_namespace)</robotNamespace> -->
+                <topicName>go2_gazebo/scan</topicName>
+                <frameName>go2_gazebo/lidar</frameName>
             </plugin>
         </sensor>
