Commit message: go2 static_tf base_gazebo

File: unitree_go2/unitree_ros/robots/go2_description/urdf/go2_description.urdf (robot description, URDF)
Before this commit: robot go2_description, 42 links, 41 joints
Links:
- removed link base
- added link base_gazebo, mass 6.921; collision box size=0.3762 0.0935 0.114; visual mesh filename=package://go2_description/dae/base.dae
Joints:
- joint FL_hip_joint: parent base -> base_gazebo
- joint FL_hip_rotor_joint: parent base -> base_gazebo
- joint FR_hip_joint: parent base -> base_gazebo
- joint FR_hip_rotor_joint: parent base -> base_gazebo
- joint Head_upper_joint: parent base -> base_gazebo
- joint RL_hip_joint: parent base -> base_gazebo
- joint RL_hip_rotor_joint: parent base -> base_gazebo
- joint RR_hip_joint: parent base -> base_gazebo
- joint RR_hip_rotor_joint: parent base -> base_gazebo
- joint front_camera_joint: parent base -> base_gazebo
- joint imu_joint: parent base -> base_gazebo
- joint radar_joint: parent base -> base_gazebo

File: unitree_go2/unitree_ros/robots/go2_description/xacro/gazebo.xacro (robot description, xacro)
@@ -13,5 +13,5 @@
             <frequency>10</frequency>
             <plot>
-                <link>base</link>
+                <link>base_gazebo</link>
                 <pose>0 0 0 0 0 0</pose>
                 <material>Gazebo/Yellow</material>
@@ -192,5 +192,5 @@
         </visual>
     </gazebo>
-    <gazebo reference="base">
+    <gazebo reference="base_gazebo">
         <turnGravityOff>false</turnGravityOff>
     </gazebo>

File: unitree_go2/unitree_ros/robots/go2_description/xacro/robot.xacro (robot description, xacro)
@@ -18,8 +18,8 @@
             <origin rpy="0 0 0" xyz="0 0 0"/>
             <parent link="world"/>
-            <child link="base"/>
+            <child link="base_gazebo"/>
         </joint>
     </xacro:if>
-    <link name="base">
+    <link name="base_gazebo">
         <visual>
             <origin rpy="0 0 0" xyz="0 0 0"/>
@@ -31,5 +31,5 @@
     <joint name="floating_base" type="fixed">
         <origin rpy="0 0 0" xyz="0 0 0"/>
-        <parent link="base"/>
+        <parent link="base_gazebo"/>
         <child link="trunk"/>
     </joint>
@@ -114,5 +114,5 @@
     </link>
     <joint name="lidar_joint" type="fixed">
-        <parent link="base" />
+        <parent link="base_gazebo" />
         <child link="lidar" />
         <origin xyz="0.23 0 0.10377" />
